File: Termo-Relay.brd (EAGLE design)
At the start: 46 x 52.1 mm, 50 parts, among them CN1 PBS-2-VERTICAL, CN2 PBS-2-VERTICAL, CN3 PBS-2-VERTICAL, CN5 PBS-4-VERTICAL, IC1 74HCT595D, IC2 74HCT595D, IC3 STM8S103FP, Q2 16M, T1 2N2222, T2 2N2222, T3 2N2222, T4 2N2222

Commit message: silk was normalized. Author was added
Routing:
- net BTN_INDIC: vias 2 -> 1
Other:
- board text added: "+"
- board text added: "-"
- board text added: "IN"
- board text added: "Polyakov Konstantin, Russia, Yeysk, 2018-05-16"
